File: main.kicad_pcb (KiCad board)
At the start: 2 copper layers, 221.6 x 89.6 mm, 122 parts, among them SW1 Kailh-Choc, SW10 Kailh-Choc, SW11 Kailh-Choc, SW12 Kailh-Choc, SW13 Kailh-Choc, SW14 Kailh-Choc, SW15 Kailh-Choc, SW16 Kailh-Choc, SW17 Kailh-Choc, SW18 Kailh-Choc, SW19 Kailh-Choc, SW2 Kailh-Choc, SW20 Kailh-Choc, SW21 Kailh-Choc, SW22 Kailh-Choc, SW23 Kailh-Choc, SW24 Kailh-Choc, SW25 Kailh-Choc, SW26 Kailh-Choc, SW27 Kailh-Choc, SW28 Kailh-Choc, SW29 Kailh-Choc, SW3 Kailh-Choc, SW30 Kailh-Choc, SW31 Kailh-Choc, SW32 Kailh-Choc, SW33 Kailh-Choc, SW34 Kailh-Choc, SW4 Kailh-Choc, SW5 Kailh-Choc, SW6 Kailh-Choc, SW7 Kailh-Choc, SW8 Kailh-Choc, SW9 Kailh-Choc, U1 nice_nano, U2 nice_nano

Commit message: try 1: cherry footprint added
* NOTE: this is not valid implementation. Footprint are fitting that
  does not mean that it will work on physical PCB. Need to redesign it.
Parts:
- removed H1 (x2), H2 (x2), H3 (x2), H4 (x4): M2 Hole, swoop:M2_hole_4.2mm
- removed REF**: OSHW-Symbol_6.7x6mm_SilkScreen, Symbol:OSHW-Symbol_6.7x6mm_SilkScreen
- removed Ref** (x4): Val**, chocolad:M2_hole_3.5mm
- removed Ref** (x4): Val**, swoop:M2_hole_3.5mm
- removed kibuzzard-63659328: G***, kibuzzard-63659328
- removed kibuzzard-63703FC3: G***, kibuzzard-63703FC3
- removed mouse-bite-2mm-slot (x2): VAL**, Duckyb-Parts:mouse-bite-5mm-slot-with-space-for-track
- SW1, SW10, SW11, SW12, SW13, SW14, SW15, SW16, SW17, SW18, SW19, SW2, SW20, SW21, SW22, SW23, SW24, SW25, SW26, SW27, SW28, SW29, SW3, SW30, SW31, SW32, SW33, SW34, SW4, SW5, SW6, SW7, SW8, SW9: footprint * duckyb-collection:SW_Hotswap_Kailh_Choc_V1_tweaked -> kbd:CherryMX_Hotswap
- moved D17 44.0 mm to (234.9, 128.7), turned to -120 degrees
- moved SW6 41.8 mm to (162.2, 95.2)
- moved D16 41.8 mm to (234.3, 123.8)
- moved SW7 41.8 mm to (180.2, 83.2)
- moved D10 41.8 mm to (239.4, 94.6)
- moved D3 41.8 mm to (206.9, 61.4)
- moved D4 41.8 mm to (225.1, 67.8)
- moved D8 41.8 mm to (207.1, 80.0)
- moved D12 41.8 mm to (188.8, 101.7)
- moved D14 41.8 mm to (224.8, 102.4)
- moved D15 41.8 mm to (239.3, 111.6)
- moved D2 41.8 mm to (188.8, 67.3)
- moved D5 41.8 mm to (239.6, 77.7)
- moved D7 41.8 mm to (188.8, 85.1)
- moved Display1 41.8 mm to (252.8, 96.7)
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- renumbered kibuzzard-636592CC to 1-kibuzzard-636592CC, G*** to 10-G***, G*** to 11-G***, REF_PUCK_R to 13-REF_PUCK_R, kibuzzard-6365950B to 2-kibuzzard-6365950B, kibuzzard-63658865 to 3-kibuzzard-63658865, kibuzzard-636588C8 to 4-kibuzzard-636588C8, kibuzzard-63659465 to 5-kibuzzard-63659465, kibuzzard-63658823 to 6-kibuzzard-63658823, kibuzzard-6361375E to 7-kibuzzard-6361375E, G*** to 9-G***
Routing:
- net COL2: track 97.7 -> 124.8 mm, vias 3 -> 0
- net R_COL4: track 134.2 -> 111.6 mm, vias 1 -> 0
- net R_COL0: track 75.2 -> 63.3 mm, vias 1 -> 0
- net Net-(D33-Pad2): track 3.46 -> 12.4 mm
- net RESET: track 47.9 -> 39.8 mm
- net R_MOSI: track 37.0 -> 29.6 mm, vias 1 -> 0
- net MOSI: track 37.3 -> 30.8 mm
- net ROW2: track 109.4 -> 115.5 mm, vias 1 -> 0
- net GND: track 66.8 -> 72.5 mm, vias 3 -> 0
- net R_GND: track 71.9 -> 66.3 mm, vias 3 -> 0
- net Net-(D21-Pad2): track 2.58 -> 7.93 mm
- net Net-(D16-Pad2): track 2.95 -> 8.02 mm
- net R_COL2: track 84.3 -> 79.2 mm
- net R_COL3: track 102.5 -> 97.5 mm, vias 1 -> 0
- net Net-(D22-Pad2): track 2.58 -> 7.42 mm
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