File: main.kicad_pcb (KiCad board)
At the start: 2 copper layers, 221.6 x 89.6 mm, 122 parts, among them SW1 Kailh-Choc, SW10 Kailh-Choc, SW11 Kailh-Choc, SW12 Kailh-Choc, SW13 Kailh-Choc, SW14 Kailh-Choc, SW15 Kailh-Choc, SW16 Kailh-Choc, SW17 Kailh-Choc, SW18 Kailh-Choc, SW19 Kailh-Choc, SW2 Kailh-Choc, SW20 Kailh-Choc, SW21 Kailh-Choc, SW22 Kailh-Choc, SW23 Kailh-Choc, SW24 Kailh-Choc, SW25 Kailh-Choc, SW26 Kailh-Choc, SW27 Kailh-Choc, SW28 Kailh-Choc, SW29 Kailh-Choc, SW3 Kailh-Choc, SW30 Kailh-Choc, SW31 Kailh-Choc, SW32 Kailh-Choc, SW33 Kailh-Choc, SW34 Kailh-Choc, SW4 Kailh-Choc, SW5 Kailh-Choc, SW6 Kailh-Choc, SW7 Kailh-Choc, SW8 Kailh-Choc, SW9 Kailh-Choc, U1 nice_nano, U2 nice_nano

Commit message: WIP: cherry mx supported added
*TODO: routing still missing
Parts:
- removed H1 (x2), H2 (x2), H3 (x2), H4 (x4): M2 Hole, swoop:M2_hole_4.2mm
- removed REF**: OSHW-Symbol_6.7x6mm_SilkScreen, Symbol:OSHW-Symbol_6.7x6mm_SilkScreen
- removed REF_PUCK_R (x2): Tenting Puck, * duckyb-collection:Tenting_Puck2_no_pads
- removed Ref** (x4): Val**, chocolad:M2_hole_3.5mm
- removed Ref** (x4): Val**, swoop:M2_hole_3.5mm
- removed kibuzzard-63659328: G***, kibuzzard-63659328
- removed kibuzzard-63703FC3: G***, kibuzzard-63703FC3
- removed mouse-bite-2mm-slot (x2): VAL**, Duckyb-Parts:mouse-bite-5mm-slot-with-space-for-track
- added 1-mouse-bite-2mm-slot: VAL**, Duckyb-Parts:mouse-bite-5mm-slot-with-space-for-track, F.Cu at (147.6, 103.8)
- added 1-mouse-bite-2mm-slot: VAL**, Duckyb-Parts:mouse-bite-5mm-slot-with-space-for-track, F.Cu at (147.6, 86.2)
- SW1, SW10, SW11, SW12, SW13, SW14, SW15, SW16, SW17, SW18, SW19, SW2, SW20, SW21, SW22, SW23, SW24, SW25, SW26, SW27, SW28, SW29, SW3, SW30, SW31, SW32, SW33, SW34, SW4, SW5, SW6, SW7, SW8, SW9: footprint * duckyb-collection:SW_Hotswap_Kailh_Choc_V1_tweaked -> marbastlib-mx:SW_MX_HS_1u; moved to B.Cu
- moved 11-kibuzzard-63658823 85.3 mm to (133.3, 123.2), turned to 0 degrees
- moved 12-kibuzzard-6361375E 84.8 mm to (133.5, 123.2), turned to 180 degrees
- moved kibuzzard-63658830 52.2 mm to (162.1, 122.9), turned to 0 degrees
- moved kibuzzard-6361375E 50.7 mm to (162.4, 122.9), turned to 180 degrees
- moved D17 49.3 mm to (237.3, 133.4)
- moved D16 48.2 mm to (233.0, 132.0)
- moved D13 47.9 mm to (207.1, 102.0)
- moved D14 46.9 mm to (226.2, 107.6)
- moved SW17 46.6 mm to (248.3, 131.8), turned to 150 degrees
- moved D12 45.8 mm to (188.1, 106.8)
- moved D34 45.4 mm to (61.5, 132.1)
- moved D33 45.4 mm to (58.0, 133.3)
- moved D15 44.7 mm to (245.2, 110.7), turned to 90 degrees
- moved D11 44.5 mm to (169.2, 117.9)
- moved D8 44.4 mm to (207.1, 82.9)
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- renumbered G*** to 1-G***, kibuzzard-636592CC to 1-kibuzzard-636592CC, kibuzzard-63658823 to 11-kibuzzard-63658823, kibuzzard-6361375E to 12-kibuzzard-6361375E, kibuzzard-63659465 to 13-kibuzzard-63659465, kibuzzard-6365950B to 2-kibuzzard-6365950B, G*** to 3-G***, kibuzzard-63658865 to 3-kibuzzard-63658865, kibuzzard-636588C8 to 4-kibuzzard-636588C8, G*** to logo-3-G***
Routing:
- net R_ROW0: track 143.4 -> 0.00 mm, vias 2 -> 0
- net COL0: track 135.7 -> 0.00 mm, vias 3 -> 0
- net R_COL4: track 134.2 -> 0.00 mm, vias 1 -> 0
- net R_ROW1: track 132.8 -> 0.00 mm, vias 3 -> 0
- net R_ROW2: track 125.7 -> 0.00 mm, vias 1 -> 0
- net ROW0: track 124.4 -> 0.00 mm, vias 2 -> 0
- net ROW1: track 115.1 -> 0.00 mm, vias 3 -> 0
- net ROW2: track 109.4 -> 0.00 mm, vias 1 -> 0
- net COL1: track 109.0 -> 0.00 mm, vias 1 -> 0
- net R_COL3: track 102.5 -> 0.00 mm, vias 1 -> 0
- net COL2: track 97.7 -> 0.00 mm, vias 3 -> 0
- net R_COL1: track 89.9 -> 0.00 mm, vias 2 -> 0
- net COL3: track 85.5 -> 0.00 mm, vias 1 -> 0
- net R_COL2: track 84.3 -> 0.00 mm, vias 1 -> 0
- net COL4: track 81.1 -> 0.00 mm, vias 2 -> 0
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- removed copper zone on B.Cu, net (none)
- removed copper zone on F.Cu, net (none)
Other:
- board size 221.6 x 89.6 mm -> 241.2 x 99.3 mm

Commit message: adding routes and zone
Parts:
- removed the 1-mouse-bite-2mm-slot at (147.6, 103.8)
- added 2-mouse-bite-2mm-slot: VAL**, Duckyb-Parts:mouse-bite-5mm-slot-with-space-for-track, F.Cu at (147.6, 103.8)
- D1, D10, D11, D12, D13, D14, D15, D16, D17, D18, D19, D2, D20, D21, D22, D23, D24, D25, D26, D27, D28, D29, D3, D30, D31, D32, D33, D34, D4, D5, D6, D7, D8, D9: footprint * duckyb-collection:SMD_Diode_Tiny -> Diode_SMD:Nexperia_CFP3_SOD-123W; moved to B.Cu
- SW1, SW10, SW11, SW12, SW13, SW14, SW15, SW16, SW17, SW18, SW19, SW2, SW20, SW21, SW22, SW23, SW24, SW25, SW26, SW27, SW28, SW29, SW3, SW30, SW31, SW32, SW33, SW34, SW4, SW5, SW6, SW7, SW8, SW9: footprint marbastlib-mx:SW_MX_HS_1u -> MX_Only:MXOnly-1U-Hotswap; moved to F.Cu
- moved SW24 38.1 mm to (115.9, 81.8), turned to 0 degrees
- moved SW26 38.1 mm to (77.8, 81.0), turned to 0 degrees
- moved D23 22.1 mm to (50.4, 77.8)
- moved D28 22.0 mm to (50.4, 96.8)
- moved D18 22.0 mm to (50.4, 58.7)
- moved D17 17.6 mm to (247.7, 119.1), turned to -30 degrees
- moved D11 17.6 mm to (151.6, 118.3)
- moved D1 17.4 mm to (151.6, 80.2)
- moved D6 17.4 mm to (151.6, 99.2)
- moved D10 17.4 mm to (227.8, 92.1)
- moved D14 17.4 mm to (208.8, 108.0)
- moved D15 17.4 mm to (227.8, 111.1)
- moved D4 17.4 mm to (208.8, 69.8)
- moved D13 17.4 mm to (189.7, 102.2)
- moved D8 17.4 mm to (189.7, 83.2)
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Routing:
- net ROW0: track 0.00 -> 204.8 mm
- net R_COL1: track 0.00 -> 189.2 mm
- net R_ROW0: track 0.00 -> 178.9 mm
- net ROW1: track 0.00 -> 158.6 mm, vias 0 -> 2
- net R_COL4: track 0.00 -> 156.7 mm
- net R_ROW1: track 0.00 -> 154.3 mm, vias 0 -> 1
- net COL0: track 0.00 -> 141.3 mm, vias 0 -> 1
- net ROW2: track 0.00 -> 129.0 mm, vias 0 -> 1
- net R_ROW2: track 0.00 -> 127.7 mm, vias 0 -> 1
- net COL1: track 0.00 -> 123.8 mm, vias 0 -> 1
- net R_COL3: track 0.00 -> 123.0 mm, vias 0 -> 3
- net COL3: track 0.00 -> 119.1 mm
- net COL4: track 0.00 -> 114.2 mm
- net R_COL2: track 0.00 -> 106.9 mm
- net COL2: track 0.00 -> 104.1 mm, vias 0 -> 1
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- added copper zone on B.Cu, net (none)
- added copper zone on F.Cu, net (none)

Commit message: minor update to PCB and name changes
Other:
- outline, holes or cut-outs redrawn
Changed lines of the file:
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@@
   (paper "A4")
   (title_block
-    (title "Urchin on Steroids")
+    (title "Ursa - Urchin on Steroids")
     (rev "v.1.0")
   )
@@
       (sketchpadsonfab false)
       (subtractmaskfromsilk false)
-      (outputformat 1)
+      (outputformat 5)
       (mirror false)
-      (drillshape 1)
+      (drillshape 0)
       (scaleselection 1)
       (outputdirectory "")
@@
   (gr_line (start 148.860169 106.299) (end 148.463 106.299) (layer "Edge.Cuts") (width 0.05))
   (gr_line (start 148.860169 106.299) (end 148.860169 120.866113) (layer "Edge.Cuts") (width 0.05))
+  (gr_line (start 252.431036 144.572711) (end 265.176 122.428) (layer "Edge.Cuts") (width 0.05))
   (gr_line (start 146.304 63.881) (end 146.304 83.680513) (layer "Edge.Cuts") (width 0.05))
   (gr_arc (start 146.320169 120.866113) (mid 146.131261 121.669384) (end 145.558169 122.263113) (layer "Edge.Cuts") (width 0.05))
   (gr_arc (start 145.558169 122.263113) (mid 129.751355 128.625656) (end 112.847803 130.772113) (layer "Edge.Cuts") (width 0.05))
   (gr_arc (start 249.047 70.542191) (mid 248.101986 70.229033) (end 247.65 69.342) (layer "Edge.Cuts") (width 0.05))
+  (gr_arc (start 182.332535 130.772113) (mid 165.428983 128.625656) (end 149.622169 122.263113) (layer "Edge.Cuts") (width 0.05))
   (gr_arc (start 148.463 101.219) (mid 147.574 101.808697) (end 146.685 101.219) (layer "Edge.Cuts") (width 0.05))
   (gr_line (start 146.304 101.219) (end 146.685 101.219) (layer "Edge.Cuts") (width 0.05))
-  (gr_arc (start 209.059148 130.772113) (mid 226.154025 133.098935) (end 242.09375 139.7) (layer "Edge.Cuts") (width 0.05))
   (gr_line (start 53.18125 139.7) (end 44.45 144.78) (layer "Edge.Cuts") (width 0.05))
   (gr_line (start 47.573589 56.884499) (end 47.573589 69.469) (layer "Edge.Cuts") (width 0.05))
   (gr_line (start 146.320169 106.299) (end 146.685 106.299) (layer "Edge.Cuts") (width 0.05))
   (gr_arc (start 44.45 144.78) (mid 43.587846 144.96327) (end 42.8625 144.4625) (layer "Edge.Cuts") (width 0.05))
+  (gr_arc (start 208.338331 130.772113) (mid 225.746285 133.058428) (end 241.999088 139.7) (layer "Edge.Cuts") (width 0.05))
   (gr_arc (start 94.377169 45.809113) (mid 121.522294 49.731191) (end 145.669 62.738) (layer "Edge.Cuts") (width 0.05))
   (gr_arc (start 148.844 63.881) (mid 149.013525 63.227292) (end 149.479 62.738) (layer "Edge.Cuts") (width 0.05))
-  (gr_arc (start 183.053352 130.772113) (mid 165.986032 128.633745) (end 150.01875 122.2375) (layer "Edge.Cuts") (width 0.05))
   (gr_line (start 30.115169 122.390113) (end 42.8625 144.4625) (layer "Edge.Cuts") (width 0.05))
   (gr_arc (start 53.18125 139.7) (mid 69.434053 133.058427) (end 86.842007 130.772113) (layer "Edge.Cuts") (width 0.05))
@@
   (gr_line (start 148.844 63.881) (end 148.844 83.693) (layer "Edge.Cuts") (width 0.05))
   (gr_arc (start 47.573589 56.884499) (mid 47.693177 56.478417) (end 48.01359 56.201738) (layer "Edge.Cuts") (width 0.05))
+  (gr_arc (start 149.622169 122.263113) (mid 149.049068 121.669395) (end 148.860169 120.866113) (layer "Edge.Cuts") (width 0.05))
   (gr_arc (start 149.479 62.738) (mid 171.224146 50.176089) (end 195.961 45.847) (layer "Edge.Cuts") (width 0.05))
-  (gr_line (start 250.698 144.78) (end 242.09375 139.7) (layer "Edge.Cuts") (width 0.05))
-  (gr_line (start 252.431036 144.572711) (end 265.176 122.428) (layer "Edge.Cuts") (width 0.05))
   (gr_arc (start 146.685 106.299) (mid 147.574 105.705003) (end 148.463 106.299) (layer "Edge.Cuts") (width 0.05))
   (gr_line (start 112.847803 130.772113) (end 86.842007 130.772113) (layer "Edge.Cuts") (width 0.05))
   (gr_line (start 27.432 70.485) (end 46.228 70.485) (layer "Edge.Cuts") (width 0.05))
-  (gr_line (start 209.059148 130.772113) (end 183.053352 130.772113) (layer "Edge.Cuts") (width 0.05))
   (gr_arc (start 195.961 45.847) (mid 222.113777 48.419233) (end 247.202529 56.238357) (layer "Edge.Cuts") (width 0.05))
-  (gr_arc (start 252.431036 144.572711) (mid 251.609177 145.04973) (end 250.698 144.78) (layer "Edge.Cuts") (width 0.05))
+  (gr_line (start 208.338331 130.772113) (end 182.332535 130.772113) (layer "Edge.Cuts") (width 0.05))
   (gr_line (start 268.223874 70.993) (end 268.224127 108.204) (layer "Edge.Cuts") (width 0.05))
+  (gr_line (start 250.730338 144.78) (end 241.999088 139.7) (layer "Edge.Cuts") (width 0.05))
   (gr_arc (start 267.589 70.485) (mid 268.011647 70.607513) (end 268.223874 70.993) (layer "Edge.Cuts") (width 0.05))
   (gr_arc (start 146.685 88.773) (mid 147.574 88.184548) (end 148.463 88.773) (layer "Edge.Cuts") (width 0.05))
+  (gr_arc (start 252.431036 144.572711) (mid 251.625346 145.042759) (end 250.730338 144.78) (layer "Edge.Cuts") (width 0.05))
   (gr_line (start 146.320169 120.866113) (end 146.320169 106.299) (layer "Edge.Cuts") (width 0.05))
   (gr_arc (start 27.051 70.866) (mid 27.162592 70.596592) (end 27.432 70.485) (layer "Edge.Cuts") (width 0.05))
   (gr_arc (start 148.463 83.693) (mid 147.569848 84.277833) (end 146.685 83.680513) (layer "Edge.Cuts") (width 0.05))
   (gr_arc (start 47.573589 69.469) (mid 47.109483 70.253367) (end 46.228 70.485) (layer "Edge.Cuts") (width 0.05))
-  (gr_arc (start 150.01875 122.2375) (mid 149.250894 121.711111) (end 148.860169 120.866113) (layer "Edge.Cuts") (width 0.05))
   (gr_line (start 148.844 88.773) (end 148.463 88.773) (layer "Edge.Cuts") (width 0.05))
   (gr_line (start 247.65 69.342) (end 247.65 56.896) (layer "Edge.Cuts") (width 0.05))
