File: main.kicad_sch (KiCad schematic)
At the start: 80 parts, among them SW1 Kailh-Choc, SW10 Kailh-Choc, SW11 Kailh-Choc, SW12 Kailh-Choc, SW13 Kailh-Choc, SW14 Kailh-Choc, SW15 Kailh-Choc, SW16 Kailh-Choc, SW17 Kailh-Choc, SW18 Kailh-Choc, SW19 Kailh-Choc, SW2 Kailh-Choc, SW20 Kailh-Choc, SW21 Kailh-Choc, SW22 Kailh-Choc, SW23 Kailh-Choc, SW24 Kailh-Choc, SW25 Kailh-Choc, SW26 Kailh-Choc, SW27 Kailh-Choc, SW28 Kailh-Choc, SW29 Kailh-Choc, SW3 Kailh-Choc, SW30 Kailh-Choc, SW31 Kailh-Choc, SW32 Kailh-Choc, SW33 Kailh-Choc, SW34 Kailh-Choc, SW4 Kailh-Choc, SW5 Kailh-Choc, SW6 Kailh-Choc, SW7 Kailh-Choc, SW8 Kailh-Choc, SW9 Kailh-Choc, U1 nice_nano, U2 nice_nano

Commit message: WIP: cherry mx supported added
*TODO: routing still missing
Parts:
- SW1, SW10, SW11, SW12, SW13, SW14, SW15, SW16, SW17, SW18, SW19, SW2, SW20, SW21, SW22, SW23, SW24, SW25, SW26, SW27, SW28, SW29, SW3, SW30, SW31, SW32, SW33, SW34, SW4, SW5, SW6, SW7, SW8, SW9: footprint * duckyb-collection:SW_Hotswap_Kailh_Choc_V1_tweaked -> marbastlib-mx:SW_MX_HS_1u; symbol MX_Alps_Hybrid:MX-NoLED -> marbastlib-mx:MX_SW_HS
Other:
- title: (none) -> Urchin on Steroids

Commit message: adding routes and zone
Parts:
- SW1, SW10, SW11, SW12, SW13, SW14, SW15, SW16, SW17, SW18, SW19, SW2, SW20, SW21, SW22, SW23, SW24, SW25, SW26, SW27, SW28, SW29, SW3, SW30, SW31, SW32, SW33, SW34, SW4, SW5, SW6, SW7, SW8, SW9: footprint marbastlib-mx:SW_MX_HS_1u -> MX_Only:MXOnly-1U-Hotswap

Commit message: minor update to PCB and name changes
Other:
- title: Urchin on Steroids -> Ursa - Urchin on Steroids
Changed lines of the file:
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@@
   (paper "A4")
   (title_block
-    (title "Urchin on Steroids")
+    (title "Ursa - Urchin on Steroids")
     (rev "v1.0")
   )
