File: ursa.kicad_sch (KiCad schematic)
At the start: 80 parts, among them SW1 Kailh-Choc, SW10 Kailh-Choc, SW11 Kailh-Choc, SW12 Kailh-Choc, SW13 Kailh-Choc, SW14 Kailh-Choc, SW15 Kailh-Choc, SW16 Kailh-Choc, SW17 Kailh-Choc, SW18 Kailh-Choc, SW19 Kailh-Choc, SW2 Kailh-Choc, SW20 Kailh-Choc, SW21 Kailh-Choc, SW22 Kailh-Choc, SW23 Kailh-Choc, SW24 Kailh-Choc, SW25 Kailh-Choc, SW26 Kailh-Choc, SW27 Kailh-Choc, SW28 Kailh-Choc, SW29 Kailh-Choc, SW3 Kailh-Choc, SW30 Kailh-Choc, SW31 Kailh-Choc, SW32 Kailh-Choc, SW33 Kailh-Choc, SW34 Kailh-Choc, SW4 Kailh-Choc, SW5 Kailh-Choc, SW6 Kailh-Choc, SW7 Kailh-Choc, SW8 Kailh-Choc, SW9 Kailh-Choc, U1 nice_nano, U2 nice_nano

Commit message: mouser bite added as library
Parts:
- added H1: Mouser Bite, extra:mouse-bite-2mm-slot-with-space-for-track, symbol Mechanical:MountingHole
- added H2: MouserBite, extra:mouse-bite-2mm-slot-with-space-for-track, symbol Mechanical:MountingHole
- D1, D10, D11, D12, D13, D14, D15, D16, D17, D18, D19, D2, D20, D21, D22, D23, D24, D25, D26, D27, D28, D29, D3, D30, D31, D32, D33, D34, D4, D5, D6, D7, D8, D9: footprint * duckyb-collection:D_SMD_TH -> Diode_SMD:D_SOD-123
- SW1, SW10, SW11, SW12, SW13, SW14, SW15, SW16, SW17, SW18, SW19, SW2, SW20, SW21, SW22, SW23, SW24, SW25, SW26, SW27, SW28, SW29, SW3, SW30, SW31, SW32, SW33, SW34, SW4, SW5, SW6, SW7, SW8, SW9: footprint MX_Only:MXOnly-1U-Hotswap -> marbastlib-mx:SW_MX_HS_1u

Commit message: library changes with new routes
Parts:
- SW_POWER0, SW_POWER1: footprint * duckyb-collection:SPDT_C128955 -> marbastlib-various:SW_MSK12C02-HB
Changed lines of the file:
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@@
     (property "Reference" "SW_POWER1" (id 0) (at 201.93 117.221 0))
     (property "Value" "SW_SPDT" (id 1) (at 201.93 119.5324 0))
-    (property "Footprint" "* duckyb-collection:SPDT_C128955" (id 2) (at 201.93 124.46 0)
+    (property "Footprint" "marbastlib-various:SW_MSK12C02-HB" (id 2) (at 201.93 124.46 0)
       (effects (font (size 1.27 1.27)) hide)
     )
@@
     (property "Reference" "SW_POWER0" (id 0) (at 201.93 27.051 0))
     (property "Value" "SW_SPDT" (id 1) (at 201.93 29.3624 0))
-    (property "Footprint" "* duckyb-collection:SPDT_C128955" (id 2) (at 201.93 34.29 0)
+    (property "Footprint" "marbastlib-various:SW_MSK12C02-HB" (id 2) (at 201.93 34.29 0)
       (effects (font (size 1.27 1.27)) hide)
     )
@@
     )
     (path "/527e5467-04a2-48e0-afae-f95895b2f459"
-      (reference "SW_POWER0") (unit 1) (value "SW_SPDT") (footprint "* duckyb-collection:SPDT_C128955")
+      (reference "SW_POWER0") (unit 1) (value "SW_SPDT") (footprint "marbastlib-various:SW_MSK12C02-HB")
     )
     (path "/3921fc0d-e37b-496e-a2dc-94330d12dbda"
-      (reference "SW_POWER1") (unit 1) (value "SW_SPDT") (footprint "* duckyb-collection:SPDT_C128955")
+      (reference "SW_POWER1") (unit 1) (value "SW_SPDT") (footprint "marbastlib-various:SW_MSK12C02-HB")
     )
     (path "/22166c71-edfc-4617-b73f-3dc820876130"
